Commit message: Created the robot urdf

File: src/oryksdog_description/urdf/macros.xacro (robot description, xacro)
@@ -1,3 +1,5 @@
 <?xml version="1.0"?>
 <robot xmlns:xacro="http://www.ros.org/wiki/xacro" name="oryksdog">
+    <!-- Maximum torque -->
+    <xacro:property name="effort_limit" value="1.4" />
 </robot>

File: src/oryksdog_description/urdf/oryksdog.xacro (robot description, xacro)
@@ -1,9 +1,787 @@
 <?xml version="1.0"?>
 <robot xmlns:xacro="http://www.ros.org/wiki/xacro" name="oryksdog">
-    <xacro:include filename="$(find oryksdog_description)/oryksdog_properties.xacro"/>
-    <xacro:include filename="$(find oryksdog_description)/macros.xacro"/>
-    <xacro:include filename="$(find oryksdog_description)/materials.xacro"/>
-    <xacro:include filename="$(find oryksdog_description)/sensors.xacro"/>
-    <xacro:include filename="$(find oryksdog_description)/gazebo_properties.xacro"/>
-    <xacro:include filename="$(find oryksdog_description)/gazebo_plugins.xacro"/>
+    <xacro:include filename="$(find oryksdog_description)/urdf/oryksdog_properties.xacro"/>
+    <xacro:include filename="$(find oryksdog_description)/urdf/macros.xacro"/>
+    <xacro:include filename="$(find oryksdog_description)/urdf/materials.xacro"/>
+    <xacro:include filename="$(find oryksdog_description)/urdf/sensors.xacro"/>
+    <xacro:include filename="$(find oryksdog_description)/urdf/gazebo_properties.xacro"/>
+    <xacro:include filename="$(find oryksdog_description)/urdf/gazebo_plugins.xacro"/>
+    <link name="base_footprint">
+    </link>
+    <joint name="fixed" type="fixed">
+        <parent link="base_footprint"/>
+        <child link="base_link"/>
+        <origin xyz="0.0 0.0 0.0" rpy="0.0 0.0 0.0"/>
+    </joint>
+    <!-- base_link -->
+    <link name="base_link">
+        <inertial>
+        <origin
+            xyz="-0.00048043 9.0814E-05 0.00023409"
+            rpy="0 0 0" />
+        <mass
+            value="0.81776" />
+        <inertia
+            ixx="0.00058474"
+            ixy="-1.0045E-06"
+            ixz="1.0886E-08"
+            iyy="0.00029699"
+            iyz="3.2027E-08"
+            izz="0.00063853" />
+        </inertial>
+        <visual>
+        <origin
+            xyz="0 0 0"
+            rpy="0 0 0" />
+        <geometry>
+            <mesh
+            filename="package://oryksdog_description/meshes/body_obj.obj" />
+        </geometry>
+        </visual>
+        <collision>
+        <origin
+            xyz="0 0 0"
+            rpy="0 0 0" />
+        <geometry>
+            <box size="0.25 0.1285 0.055"/>
+        </geometry>
+        </collision>
+    </link>
+    <!--Front Right Leg Links-->
+    <!-- FR1 -->
+    <link name="FR1">
+        <inertial>
+        <origin
+            xyz="0.011092 -0.0032719 0.00019267"
+            rpy="0 0 0" />
+        <mass
+            value="0.15379" />
+        <inertia
+            ixx="4.474E-05"
+            ixy="-1.0746E-05"
+            ixz="-1.7651E-07"
+            iyy="4.3489E-05"
+            iyz="-7.8105E-08"
+            izz="6.8646E-05" />
+        </inertial>
+        <visual>
+        <origin
+            xyz="0 0 0"
+            rpy="0 0 0" />
+        <geometry>
+            <mesh
+            filename="package://oryksdog_description/meshes/FR1_obj.obj" />
+        </geometry>
+        </visual>
+    </link>
+    <!-- FR2 -->
+    <link name="FR2">
+        <inertial>
+        <origin
+            xyz="0.038603 -0.0025578 -0.0001752"
+            rpy="0 0 0" />
+        <mass
+            value="0.15106" />
+        <inertia
+            ixx="2.365E-05"
+            ixy="-5.3771E-07"
+            ixz="-1.6144E-06"
+            iyy="0.00010469"
+            iyz="8.3059E-08"
+            izz="0.00011187" />
+        </inertial>
+        <visual>
+        <origin
+            xyz="0 0 0"
+            rpy="0 0 0" />
+        <geometry>
+            <mesh
+            filename="package://oryksdog_description/meshes/R2_obj.obj" />
+        </geometry>
+        </visual>
+        <collision>
+        <origin
+            xyz="0.04 0 0"
+            rpy="0 1.57075 0" />
+        <geometry>
+            <cylinder length="0.125" radius="0.014"/>
+        </geometry>
+        </collision>
+    </link>
+    <!-- FR3 -->
+    <link name="FR3">
+        <inertial>
+        <origin
+            xyz="0.029797 -0.00098828 -9.2749E-05"
+            rpy="0 0 0" />
+        <mass
+            value="0.023372" />
+        <inertia
+            ixx="6.565E-07"
+            ixy="6.8071E-07"
+            ixz="-1.0503E-07"
+            iyy="2.7257E-05"
+            iyz="3.918E-09"
+            izz="2.7469E-05" />
+        </inertial>
+        <visual>
+        <origin
+            xyz="0 0 0"
+            rpy="0 0 0" />
+        <geometry>
+            <mesh
+            filename="package://oryksdog_description/meshes/R3_obj.obj" />
+        </geometry>
+        </visual>
+        <collision>
+        <origin
+            xyz="0.045 0 0"
+            rpy="0 1.57075 0" />
+        <geometry>
+            <cylinder length="0.06" radius="0.007"/>
+        </geometry>
+        </collision>
+    </link>
+    <!-- FR4 -->
+    <link name="FR4">
+        <inertial>
+        <origin
+            xyz="0.00 0 0"
+            rpy="0 0 0" />
+        <mass
+            value="0.0391" />
+        <inertia
+            ixx="3.7713E-012"
+            ixy="0"
+            ixz="0"
+            iyy="3.5422E-12"
+            iyz="0"
+            izz="5.443E-012" />
+        </inertial>
+        <collision>
+        <origin
+            xyz="0 0 0"
+            rpy="0 0 0" />
+        <geometry>
+            <sphere radius="0.0072"/>
+        </geometry>
+        </collision>
+    </link>
+    <!--Front Left Leg Links-->
+    <!-- FL1 -->
+    <link name="FL1">
+        <inertial>
+        <origin
+            xyz="-0.011124 -0.0032814 0.00014476"
+            rpy="0 0 0" />
+        <mass
+            value="0.15334" />
+        <inertia
+            ixx="4.4732E-05"
+            ixy="1.0746E-05"
+            ixz="1.7651E-07"
+            iyy="4.3482E-05"
+            iyz="-7.8105E-08"
+            izz="6.8645E-05" />
+        </inertial>
+        <visual>
+        <origin
+            xyz="0 0 0"
+            rpy="0 0 0" />
+        <geometry>
+            <mesh
+            filename="package://oryksdog_description/meshes/FL1_obj.obj" />
+        </geometry>
+        </visual>
+    </link>
+    <!-- FL2 -->
+    <link name="FL2">
+        <inertial>
+        <origin
+            xyz="0.038603 -0.0025578 0.0001752"
+            rpy="0 0 0" />
+        <mass
+            value="0.15106" />
+        <inertia
+            ixx="2.365E-05"
+            ixy="-5.3771E-07"
+            ixz="1.6144E-06"
+            iyy="0.00010469"
+            iyz="-8.306E-08"
+            izz="0.00011187" />
+        </inertial>
+        <visual>
+        <origin
+            xyz="0 0 0"
+            rpy="0 0 0" />
+        <geometry>
+            <mesh
+            filename="package://oryksdog_description/meshes/L2_obj.obj" />
+        </geometry>
+        </visual>
+        <collision>
+        <origin
+            xyz="0.04 0 0"
+            rpy="0 1.57075 0" />
+        <geometry>
+            <cylinder length="0.125" radius="0.014"/>
+        </geometry>
+        </collision>
+    </link>
+        <!-- FL3 -->
+    <link name="FL3">
+        <inertial>
+        <origin
+            xyz="0.029797 -0.0009883 9.2751E-05"
+            rpy="0 0 0" />
+        <mass
+            value="0.023372" />
+        <inertia
+            ixx="6.565E-07"
+            ixy="6.8071E-07"
+            ixz="1.0503E-07"
+            iyy="2.7257E-05"
+            iyz="-3.918E-09"
+            izz="2.7469E-05" />
+        </inertial>
+        <visual>
+        <origin
+            xyz="0 0 0"
+            rpy="0 0 0" />
+        <geometry>
+            <mesh
+            filename="package://oryksdog_description/meshes/L3_obj.obj" />
+        </geometry>
+        </visual>
+        <collision>
+        <origin
+            xyz="0.045 0 0"
+            rpy="0 1.57075 0" />
+        <geometry>
+            <cylinder length="0.06" radius="0.007"/>
+        </geometry>
+        </collision>
+    </link>
+        <!-- FL4 -->
+    <link name="FL4">
+        <inertial>
+        <origin
+            xyz="0.00 0 0"
+            rpy="0 0 0" />
+        <mass
+            value="0.0391" />
+        <inertia
+            ixx="3.7713E-012"
+            ixy="0"
+            ixz="0"
+            iyy="3.5422E-12"
+            iyz="0"
+            izz="5.443E-012" />
+        </inertial>
+        <collision>
+        <origin
+            xyz="0 0 0"
+            rpy="0 0 0" />
+        <geometry>
+            <sphere radius="0.0072"/>
+        </geometry>
+        </collision>
+    </link>
+    <!--Rear Right Leg Links-->
+    <!-- RR1 -->
+    <link name="RR1">
+        <inertial>
+        <origin
+            xyz="0.011092 -0.0032719 -0.00019266"
+            rpy="0 0 0" />
+        <mass
+            value="0.15379" />
+        <inertia
+            ixx="4.474E-05"
+            ixy="-1.0746E-05"
+            ixz="1.7651E-07"
+            iyy="4.3489E-05"
+            iyz="7.8105E-08"
+            izz="6.8646E-05" />
+        </inertial>
+        <visual>
+        <origin
+            xyz="0 0 0"
+            rpy="0 0 0" />
+        <geometry>
+            <mesh
+            filename="package://oryksdog_description/meshes/RR1_obj.obj" />
+        </geometry>
+        </visual>
+    </link>
+    <!-- RR2 -->
+    <link name="RR2">
+        <inertial>
+        <origin
+            xyz="0.038603 -0.0025578 -0.0001752"
+            rpy="0 0 0" />
+        <mass
+            value="0.15106" />
+        <inertia
+            ixx="2.365E-05"
+            ixy="-5.3771E-07"
+            ixz="-1.6144E-06"
+            iyy="0.00010469"
+            iyz="8.3059E-08"
+            izz="0.00011187" />
+        </inertial>
+        <visual>
+        <origin
+            xyz="0 0 0"
+            rpy="0 0 0" />
+        <geometry>
+            <mesh
+            filename="package://oryksdog_description/meshes/R2_obj.obj" />
+        </geometry>
+        </visual>
+        <collision>
+        <origin
+            xyz="0.04 0 0"
+            rpy="0 1.57075 0" />
+        <geometry>
+            <cylinder length="0.125" radius="0.014"/>
+        </geometry>
+        </collision>
+    </link>
+    <!-- RR3 -->
+    <link name="RR3">
+        <inertial>
+        <origin
+            xyz="0.029797 -0.00098828 -9.2749E-05"
+            rpy="0 0 0" />
+        <mass
+            value="0.023372" />
+        <inertia
+            ixx="6.565E-07"
+            ixy="6.8071E-07"
+            ixz="-1.0503E-07"
+            iyy="2.7257E-05"
+            iyz="3.918E-09"
+            izz="2.7469E-05" />
+        </inertial>
+        <visual>
+        <origin
+            xyz="0 0 0"
+            rpy="0 0 0" />
+        <geometry>
+            <mesh
+            filename="package://oryksdog_description/meshes/R3_obj.obj" />
+        </geometry>
+        </visual>
+        <collision>
+        <origin
+            xyz="0.045 0 0"
+            rpy="0 1.57075 0" />
+        <geometry>
+            <cylinder length="0.06" radius="0.007"/>
+        </geometry>
+        </collision>
+    </link>
+    <!-- RR4 -->
+    <link name="RR4">
+        <inertial>
+        <origin
+            xyz="0.00 0 0"
+            rpy="0 0 0" />
+        <mass
+            value="0.0391" />
+        <inertia
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
Commit message: Added and disabled the rplidar

File: src/oryksdog_description/urdf/macros.xacro (robot description, xacro)
@@ -1,5 +1,9 @@
 <?xml version="1.0"?>
 <robot xmlns:xacro="http://www.ros.org/wiki/xacro" name="oryksdog">
-    <!-- Maximum torque -->
-    <xacro:property name="effort_limit" value="1.4" />
+  <xacro:macro name="box_inertia" params="m w h d">
+    <inertial>
+      <mass value="${m}"/>
+      <inertia ixx="${m / 12.0 * (d*d + h*h)}" ixy="0.0" ixz="0.0" iyy="${m / 12.0 * (w*w + h*h)}" iyz="0.0" izz="${m / 12.0 * (w*w + d*d)}"/>
+    </inertial>
+  </xacro:macro>
 </robot>

File: src/oryksdog_description/urdf/materials.xacro (robot description, xacro)
@@ -1,3 +1,15 @@
 <?xml version="1.0"?>
 <robot xmlns:xacro="http://www.ros.org/wiki/xacro" name="oryksdog">
+    <material name="blue">
+	    <color rgba="0 0 0.8 1"/>
+    </material>
+    <material name="white">
+	    <color rgba="1 1 1 1"/>
+    </material>
+    <material name="black">
+	    <color rgba="0 0 0 1"/>
+    </material>
+    <material name="green">
+        <color rgba="0.0 0.8 0.0 1.0"/>
+    </material>
 </robot>

File: src/oryksdog_description/urdf/oryksdog.xacro (robot description, xacro)
@@ -4,5 +4,5 @@
     <xacro:include filename="$(find oryksdog_description)/urdf/macros.xacro"/>
     <xacro:include filename="$(find oryksdog_description)/urdf/materials.xacro"/>
-    <xacro:include filename="$(find oryksdog_description)/urdf/sensors.xacro"/>
+    <!--xacro:include filename="$(find oryksdog_description)/urdf/sensors.xacro"/-->
     <xacro:include filename="$(find oryksdog_description)/urdf/gazebo_properties.xacro"/>
     <xacro:include filename="$(find oryksdog_description)/urdf/gazebo_plugins.xacro"/>

File: src/oryksdog_description/urdf/oryksdog_properties.xacro (robot description, xacro)
@@ -1,3 +1,7 @@
 <?xml version="1.0"?>
 <robot xmlns:xacro="http://www.ros.org/wiki/xacro" name="oryksdog">
+    <!-- Maximum torque -->
+    <xacro:property name="effort_limit" value="1.4" />
+    <xacro:property name="laser_width" value="0.05"/>
+    <xacro:property name="laser_len" value="0.05"/>
 </robot>

File: src/oryksdog_description/urdf/sensors.xacro (robot description, xacro)
@@ -1,3 +1,24 @@
 <?xml version="1.0"?>
 <robot xmlns:xacro="http://www.ros.org/wiki/xacro" name="oryksdog">
+    <joint name="laser_joint" type="fixed">
+        <origin xyz="0 0.040 0.090" rpy="0 0 1.5708" />
+        <parent link="base_link" />
+        <child link="laser" />
+    </joint>
+    <link name="laser">
+    <xacro:box_inertia m="0.5" w="${laser_len}" h="${laser_width}" d="0.05"/>
+    <visual>
+      <origin rpy="0 0 -1.5708" xyz="0.084 -0.242 -0.098"/>
+      <geometry>
+        <mesh filename="package://oryksdog_description/meshes/RpLidar.stl" scale="0.001 0.001 0.001"/>
+      </geometry>
+      <material name="blue"/>
+    </visual>
+    <collision>
+      <origin rpy="0 0 0" xyz="0.242 0.084 -0.098"  />
+      <geometry>
+        <mesh filename="package://oryksdog_description/meshes/RpLidar.stl" scale="0.001 0.001 0.001" />
+      </geometry>
+    </collision>
+    </link>
 </robot>
